File: MKR-I2C-shield.brd (EAGLE design)
At the start: 25 x 61.5 mm, 45 parts, among them J1 C-GRID-04-70543, J10 DNP, J1H C-GRID-04-70553, J2 C-GRID-04-70543, J2H C-GRID-04-70553, J3 C-GRID-04-70543, J3H C-GRID-04-70553, J4 C-GRID-04-70553, J5 C-GRID-04-70543, J6 C-GRID-04-70543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

Commit message: v1.0
first production run
Parts:
- moved J2H 0.38 mm to (19.1, 47.4)
- moved J3H 0.38 mm to (6.35, 47.4)
Routing:
- net VREF_B: track 4.58 -> 5.20 mm
Other:
- board text added: "GND"
- board text added: "SCL"
- board text added: "SDA"
- board text added: "V1.0"
- board text added: "VCC"
- board text removed: "V0.1"
