File: MKR-I2C-shield.sch (EAGLE design)
At the start: 45 parts, among them J1 C-GRID-04-70543, J10 DNP, J1H C-GRID-04-70553, J2 C-GRID-04-70543, J2H C-GRID-04-70553, J3 C-GRID-04-70543, J3H C-GRID-04-70553, J4 C-GRID-04-70553, J5 C-GRID-04-70543, J6 C-GRID-04-70543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

Commit message: v1.0
first production run
Other:
- note added: "V1.0"
- note removed: "V0.1"
Changed lines of the file:
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@@
 DAMAGES OR OTHER LIABILITY, WHETHER IN AN ACTION OF CONTRACT, TORT OR OTHERWISE, ARISING FROM,
 OUT OF OR IN CONNECTION WITH THE PRODUCT OR THE USE OR OTHER DEALINGS IN THE PRODUCT.</text>
-<text x="314.96" y="12.7" size="6.4516" layer="94">V0.1</text>
+<text x="314.96" y="12.7" size="6.4516" layer="94">V1.0</text>
 </plain>
 <instances>
